Commit message: IK is working pretty smoothly. Z is clipped to base_height. The joint limits in the urdf are modified.

File: urdf/2linkarm.urdf (robot description, URDF)
Before this commit: robot 2linkarm, 4 links, 3 joints
Joints:
- joint baseHinge: limit lower=0 upper=6.28 effort=100.0 velocity=5.0 -> lower=-3.14159 upper=3.14159 effort=100.0 velocity=5.0
