Commit message: Made changes to approach in MPC (fixed time MPC)

File: urdf/3dof_planar_slider.urdf (robot description, URDF)
Before this commit: robot 3dof_planar_slider, 5 links, 4 joints
Links:
- link endEffector: mass 0.01 -> 0.1; geometry collision cylinder length=0.02 radius=0.25; visual cylinder length=0.02 radius=0.1
Joints:
- joint baseHinge: limit lower=0 upper=3.14159 effort=200.0 velocity=5.0 -> lower=-6.28 upper=6.28 effort=200.0 velocity=5.0
